File: Module schematics/Module scheme.sch (EAGLE design)
At the start: 36 parts, among them IC1 MAX7219CNG, U1 328P, U2 328P

Commit message: Added maze module schematics
Parts:
- added C1: (no value), adafruit:C-US025-024X044
- added C2: (no value), adafruit:CPOL-US085CS-1AR
- added IC2: MAX7219CNG, maxim:MAX7219CNG
- added LED11, LED12, LED13, LED14, LED15, LED16, LED17, LED18, LED19, LED20, LED21, LED22, LED23, LED24, LED25, LED26, LED27, LED28, LED29, LED30, LED31, LED32, LED33, LED34, LED35, LED36, LED37, LED38, LED39, LED40, LED41, LED42, LED43, LED44, LED45, LED46, LED47, LED48, LED49, LED50, LED51, LED52, LED53, LED54, LED55, LED56, LED57, LED58, LED59, LED60, LED61, LED62, LED63, LED64, LED65, LED66, LED67, LED68, LED69, LED70, LED71, LED72, LED73, LED74: (no value), Fidget Spinner Example:LEDCHIP-LED0805
- added R15: (no value), adafruit:R-US_0309/12
- added U3: 328P, SparkFun-IC-Microcontroller:ATMEGA328P_PDIP
Connections:
- new net N$36: IC2.SEGDP, LED67.A, LED68.A, LED69.A, LED70.A, LED71.A, LED72.A, LED73.A, LED74.A
- new net N$40: IC2.SEGA, LED59.A, LED60.A, LED61.A, LED62.A, LED63.A, LED64.A, LED65.A, LED66.A
- new net N$41: IC2.SEGB, LED51.A, LED52.A, LED53.A, LED54.A, LED55.A, LED56.A, LED57.A, LED58.A
- new net N$42: IC2.SEGC, LED43.A, LED44.A, LED45.A, LED46.A, LED47.A, LED48.A, LED49.A, LED50.A
- new net N$49: IC2.DIG0, LED11.C, LED19.C, LED27.C, LED35.C, LED43.C, LED51.C, LED59.C, LED67.C
- new net N$50: IC2.SEGE, LED27.A, LED28.A, LED29.A, LED30.A, LED31.A, LED32.A, LED33.A, LED34.A
- new net N$51: IC2.SEGF, LED19.A, LED20.A, LED21.A, LED22.A, LED23.A, LED24.A, LED25.A, LED26.A
- new net N$52: IC2.SEGD, LED35.A, LED36.A, LED37.A, LED38.A, LED39.A, LED40.A, LED41.A, LED42.A
- new net N$53: IC2.SEGG, LED11.A, LED12.A, LED13.A, LED14.A, LED15.A, LED16.A, LED17.A, LED18.A
- new net N$54: IC2.DIG1, LED12.C, LED20.C, LED28.C, LED36.C, LED44.C, LED52.C, LED60.C, LED68.C
- new net N$55: IC2.DIG2, LED13.C, LED21.C, LED29.C, LED37.C, LED45.C, LED53.C, LED61.C, LED69.C
- new net N$56: IC2.DIG3, LED14.C, LED22.C, LED30.C, LED38.C, LED46.C, LED54.C, LED62.C, LED70.C
- new net N$57: IC2.DIG4, LED15.C, LED23.C, LED31.C, LED39.C, LED47.C, LED55.C, LED63.C, LED71.C
- new net N$58: IC2.DIG5, LED16.C, LED24.C, LED32.C, LED40.C, LED48.C, LED56.C, LED64.C, LED72.C
- new net N$59: IC2.DIG6, LED17.C, LED25.C, LED33.C, LED41.C, LED49.C, LED57.C, LED65.C, LED73.C
- new net N$60: IC2.DIG7, LED18.C, LED26.C, LED34.C, LED42.C, LED50.C, LED58.C, LED66.C, LED74.C
- new net N$61: IC2.ISET, R15.1
- new net N$62: C1.1, C2.+, IC2.VCC, R15.2, U3.VCC
- new net N$63: IC2.DIN, U3.PB4(MISO)
- new net N$64: IC2.CLK, U3.PB3(MOSI/OC2)
- new net N$65: IC2.LOAD, U3.PB2(SS/OC1B)
- new net N$66: C1.2, C2.-, IC2.GND@1, IC2.GND@2, U3.GND@2
