File: Modules/Button/ECAD/Button.sch (KiCad schematic (older format))
At the start: 26 parts, among them J1 comm_header, J2 prog_header, SW1 BIG_BTN, U1 ATmega328-PU, U2 MAX7219, U3 HDSP-7503

Commit message: Added polyfuses to all modules
Parts:
- added F1: Polyfuse, symbol Device:Polyfuse
Connections:
- net VCC: now also F1.1; no longer J1.4 (Pin_4), J2.1 (Pin_1)
- new net UVCC: F1.2, J1.4 (Pin_4), J2.1 (Pin_1)
Changed lines of the file:
@@
 L power:VCC #PWR01
 U 1 1 5F5DC5B2
-P 1400 3350
-F 0 "#PWR01" H 1400 3200 50  0001 C CNN
-F 1 "VCC" V 1418 3477 50  0000 L CNN
-F 2 "" H 1400 3350 50  0001 C CNN
-F 3 "" H 1400 3350 50  0001 C CNN
-	1    1400 3350
-	0    -1   -1   0
-$EndComp
-$Comp
-L power:VCC #PWR03
-U 1 1 5F675D83
-P 1400 3950
-F 0 "#PWR03" H 1400 3800 50  0001 C CNN
-F 1 "VCC" V 1418 4077 50  0000 L CNN
-F 2 "" H 1400 3950 50  0001 C CNN
-F 3 "" H 1400 3950 50  0001 C CNN
-	1    1400 3950
-	0    -1   -1   0
+P 2400 3050
+F 0 "#PWR01" H 2400 2900 50  0001 C CNN
+F 1 "VCC" V 2418 3177 50  0000 L CNN
+F 2 "" H 2400 3050 50  0001 C CNN
+F 3 "" H 2400 3050 50  0001 C CNN
+	1    2400 3050
+	0    1    1    0
 $EndComp
 $Comp
@@
 NoConn ~ 6800 2950
 NoConn ~ 4400 2050
+$Comp
+L Device:Polyfuse F1
+U 1 1 5F928138
+P 2150 3050
+F 0 "F1" V 1925 3050 50  0000 C CNN
+F 1 "Polyfuse" V 2016 3050 50  0000 C CNN
+F 2 "" H 2200 2850 50  0001 L CNN
+F 3 "~" H 2150 3050 50  0001 C CNN
+	1    2150 3050
+	0    1    1    0
+$EndComp
+Wire Wire Line
+	2300 3050 2400 3050
+Wire Wire Line
+	1900 3050 2000 3050
+Text Label 1900 3050 2    50   ~ 0
+UVCC
+Text Label 1400 3350 2    50   ~ 0
+UVCC
+Text Label 1400 3950 2    50   ~ 0
+UVCC
 $EndSCHEMATC
