File: Modules/Maze/ECAD/Maze.sch (KiCad schematic (older format))
At the start: 10 parts, among them J1 comm_header, J2 prog_header, SW1 SW_Push_Dual_x2, SW2 SW_Push_Dual_x2, U2 ATmega328-PU

Commit message: Added polyfuses to all modules
Parts:
- added F1: Polyfuse, symbol Device:Polyfuse
Connections:
- net VCC: now also F1.1; no longer J1.4 (Pin_4), J2.1 (Pin_1)
- new net UVCC: F1.2, J1.4 (Pin_4), J2.1 (Pin_1)
Changed lines of the file:
@@
-$EndComp
-$Comp
-L power:VCC #PWR011
-U 1 1 5F6DBC0D
-P 1400 3950
-F 0 "#PWR011" H 1400 3800 50  0001 C CNN
-F 1 "VCC" V 1418 4077 50  0000 L CNN
-F 2 "" H 1400 3950 50  0001 C CNN
-F 3 "" H 1400 3950 50  0001 C CNN
-	1    1400 3950
-	0    -1   -1   0
 $EndComp
 $Comp
 L power:VCC #PWR08
 U 1 1 5F5DC5B2
-P 1400 3350
-F 0 "#PWR08" H 1400 3200 50  0001 C CNN
-F 1 "VCC" V 1418 3477 50  0000 L CNN
-F 2 "" H 1400 3350 50  0001 C CNN
-F 3 "" H 1400 3350 50  0001 C CNN
-	1    1400 3350
-	0    -1   -1   0
+P 2300 3050
+F 0 "#PWR08" H 2300 2900 50  0001 C CNN
+F 1 "VCC" V 2318 3177 50  0000 L CNN
+F 2 "" H 2300 3050 50  0001 C CNN
+F 3 "" H 2300 3050 50  0001 C CNN
+	1    2300 3050
+	0    1    1    0
 $EndComp
 $Comp
@@
 Wire Wire Line
 	4400 5700 4400 5550
+$Comp
+L Device:Polyfuse F1
+U 1 1 5F9201CD
+P 2050 3050
+F 0 "F1" V 1825 3050 50  0000 C CNN
+F 1 "Polyfuse" V 1916 3050 50  0000 C CNN
+F 2 "" H 2100 2850 50  0001 L CNN
+F 3 "~" H 2050 3050 50  0001 C CNN
+	1    2050 3050
+	0    1    1    0
+$EndComp
+Wire Wire Line
+	2300 3050 2200 3050
+Wire Wire Line
+	1800 3050 1900 3050
+Text Label 1800 3050 2    50   ~ 0
+UVCC
+Text Label 1400 3350 2    50   ~ 0
+UVCC
+Text Label 1400 3950 2    50   ~ 0
+UVCC
 $EndSCHEMATC
