File: Modules/Memory/ECAD/Memory.sch (KiCad schematic (older format))
At the start: 23 parts, among them J1 comm_header, J2 prog_header, SW1 SW_Push_Dual_x2, SW2 SW_Push_Dual_x2, U1 ATmega328-PU, U2 KCSC02-105, U3 KCSC02-105, U4 MAX7219, U5 KCSC02-105, U6 KCSC02-105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

Commit message: Added polyfuses to all modules
Parts:
- added F1: Polyfuse, symbol Device:Polyfuse
Connections:
- net VCC: now also F1.1; no longer J1.4 (Pin_4), J2.1 (Pin_1)
- new net UVCC: F1.2, J1.4 (Pin_4), J2.1 (Pin_1)
Changed lines of the file:
@@
 L power:VCC #PWR01
 U 1 1 5F5DC5B2
-P 1400 3350
-F 0 "#PWR01" H 1400 3200 50  0001 C CNN
-F 1 "VCC" V 1418 3477 50  0000 L CNN
-F 2 "" H 1400 3350 50  0001 C CNN
-F 3 "" H 1400 3350 50  0001 C CNN
-	1    1400 3350
-	0    -1   -1   0
-$EndComp
-$Comp
-L power:VCC #PWR03
-U 1 1 5F6DE2D5
-P 1400 3950
-F 0 "#PWR03" H 1400 3800 50  0001 C CNN
-F 1 "VCC" V 1418 4077 50  0000 L CNN
-F 2 "" H 1400 3950 50  0001 C CNN
-F 3 "" H 1400 3950 50  0001 C CNN
-	1    1400 3950
-	0    -1   -1   0
+P 2200 3050
+F 0 "#PWR01" H 2200 2900 50  0001 C CNN
+F 1 "VCC" V 2218 3177 50  0000 L CNN
+F 2 "" H 2200 3050 50  0001 C CNN
+F 3 "" H 2200 3050 50  0001 C CNN
+	1    2200 3050
+	0    1    1    0
 $EndComp
 $Comp
@@
 Wire Wire Line
 	8200 3450 8200 5250
+$Comp
+L Device:Polyfuse F1
+U 1 1 5F924F2E
+P 1950 3050
+F 0 "F1" V 1725 3050 50  0000 C CNN
+F 1 "Polyfuse" V 1816 3050 50  0000 C CNN
+F 2 "" H 2000 2850 50  0001 L CNN
+F 3 "~" H 1950 3050 50  0001 C CNN
+	1    1950 3050
+	0    1    1    0
+$EndComp
+Text Label 1400 3950 2    50   ~ 0
+UVCC
+Text Label 1400 3350 2    50   ~ 0
+UVCC
+Text Label 1700 3050 2    50   ~ 0
+UVCC
+Wire Wire Line
+	1700 3050 1800 3050
+Wire Wire Line
+	2100 3050 2200 3050
 $EndSCHEMATC
