File: Modules/SimonSays/ECAD/SimonSays.sch (KiCad schematic (older format))
At the start: 13 parts, among them J1 comm_header, J2 prog_header, SW1 SW_Push_LED, SW2 SW_Push_LED, SW3 SW_Push_LED, SW4 SW_Push_LED, U1 ATmega328-PU

Commit message: Added polyfuses to all modules
Parts:
- added F1: Polyfuse, symbol Device:Polyfuse
Connections:
- net VCC: now also F1.1; no longer J1.4 (Pin_4), J2.1 (Pin_1)
- new net UVCC: F1.2, J1.4 (Pin_4), J2.1 (Pin_1)
Changed lines of the file:
@@
 L power:VCC #PWR01
 U 1 1 5F5DC5B2
-P 1400 3350
-F 0 "#PWR01" H 1400 3200 50  0001 C CNN
-F 1 "VCC" V 1418 3477 50  0000 L CNN
-F 2 "" H 1400 3350 50  0001 C CNN
-F 3 "" H 1400 3350 50  0001 C CNN
-	1    1400 3350
-	0    -1   -1   0
-$EndComp
-$Comp
-L power:VCC #PWR03
-U 1 1 5F5DD568
-P 1400 3950
-F 0 "#PWR03" H 1400 3800 50  0001 C CNN
-F 1 "VCC" V 1418 4077 50  0000 L CNN
-F 2 "" H 1400 3950 50  0001 C CNN
-F 3 "" H 1400 3950 50  0001 C CNN
-	1    1400 3950
-	0    -1   -1   0
+P 2250 3100
+F 0 "#PWR01" H 2250 2950 50  0001 C CNN
+F 1 "VCC" V 2268 3227 50  0000 L CNN
+F 2 "" H 2250 3100 50  0001 C CNN
+F 3 "" H 2250 3100 50  0001 C CNN
+	1    2250 3100
+	0    1    1    0
 $EndComp
 $Comp
@@
 NoConn ~ 4400 4050
 NoConn ~ 4400 4150
+$Comp
+L Device:Polyfuse F1
+U 1 1 5F9202C9
+P 2000 3100
+F 0 "F1" V 1775 3100 50  0000 C CNN
+F 1 "Polyfuse" V 1866 3100 50  0000 C CNN
+F 2 "" H 2050 2900 50  0001 L CNN
+F 3 "~" H 2000 3100 50  0001 C CNN
+	1    2000 3100
+	0    1    1    0
+$EndComp
+Text Label 1400 3950 2    50   ~ 0
+UVCC
+Text Label 1400 3350 2    50   ~ 0
+UVCC
+Text Label 1750 3100 2    50   ~ 0
+UVCC
+Wire Wire Line
+	1750 3100 1850 3100
+Wire Wire Line
+	2150 3100 2250 3100
 $EndSCHEMATC
