File: Modules/ComplicatedWires/ECAD/ComplicatedWires.sch (KiCad schematic (older format))
At the start: 42 parts, among them J1 comm_header, J10 Conn_01x01_Female, J11 Conn_01x01_Female, J12 Conn_01x01_Female, J13 Conn_01x01_Female, J14 Conn_01x01_Female, J2 prog_header, J3 Conn_01x01_Female, J4 Conn_01x01_Female, J5 Conn_01x01_Female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

Commit message: Added polyfuses to all modules
Parts:
- added F1: Polyfuse, symbol Device:Polyfuse
Connections:
- net VCC: now also F1.1; no longer J1.4 (Pin_4), J2.1 (Pin_1)
- new net UVCC: F1.2, J1.4 (Pin_4), J2.1 (Pin_1)
Changed lines of the file:
@@
 L power:VCC #PWR01
 U 1 1 5F5DC5B2
-P 1400 3350
-F 0 "#PWR01" H 1400 3200 50  0001 C CNN
-F 1 "VCC" V 1418 3477 50  0000 L CNN
-F 2 "" H 1400 3350 50  0001 C CNN
-F 3 "" H 1400 3350 50  0001 C CNN
-	1    1400 3350
-	0    -1   -1   0
-$EndComp
-$Comp
-L power:VCC #PWR03
-U 1 1 5F5DD568
-P 1400 3950
-F 0 "#PWR03" H 1400 3800 50  0001 C CNN
-F 1 "VCC" V 1418 4077 50  0000 L CNN
-F 2 "" H 1400 3950 50  0001 C CNN
-F 3 "" H 1400 3950 50  0001 C CNN
-	1    1400 3950
-	0    -1   -1   0
+P 2300 3050
+F 0 "#PWR01" H 2300 2900 50  0001 C CNN
+F 1 "VCC" V 2318 3177 50  0000 L CNN
+F 2 "" H 2300 3050 50  0001 C CNN
+F 3 "" H 2300 3050 50  0001 C CNN
+	1    2300 3050
+	0    1    1    0
 $EndComp
 $Comp
@@
 Wire Wire Line
 	7650 2700 7800 2700
+$Comp
+L Device:Polyfuse F1
+U 1 1 5F924A65
+P 2050 3050
+F 0 "F1" V 1825 3050 50  0000 C CNN
+F 1 "Polyfuse" V 1916 3050 50  0000 C CNN
+F 2 "" H 2100 2850 50  0001 L CNN
+F 3 "~" H 2050 3050 50  0001 C CNN
+	1    2050 3050
+	0    1    1    0
+$EndComp
+Text Label 1400 3350 2    50   ~ 0
+UVCC
+Text Label 1400 3950 2    50   ~ 0
+UVCC
+Text Label 1800 3050 2    50   ~ 0
+UVCC
+Wire Wire Line
+	1800 3050 1900 3050
+Wire Wire Line
+	2200 3050 2300 3050
 $EndSCHEMATC

Commit message: Updated value of Rset for MAX7219
Parts:
- RSet1: value 27k -> 24.3
Changed lines of the file:
@@
 AR Path="/5F6805C3" Ref="RSet1"  Part="1"
 F 0 "RSet1" H 5718 3946 50  0000 L CNN
-F 1 "27k" H 5718 3855 50  0000 L CNN
+F 1 "24.3" H 5718 3855 50  0000 L CNN
 F 2 "" V 5690 3890 50  0001 C CNN
 F 3 "~" H 5650 3900 50  0001 C CNN
