File: Case/Edgework/SerialNumber/ECAD/EPaperDriver.kicad_pcb (KiCad board)
At the start: 4 copper layers, 89.5 x 38 mm, 32 parts, among them J1 Micro_SD_Card_Det, J2 Conn_01x11, Q1 Si1304BDL, U1 TXS0108EPW, U2 RT9193-33GB, U3 23LC1024

Commit message: Moved some files into correct subfolder
Parts:
- J2: value Conn_01x11 -> Conn_01x12; footprint Connector_PinHeader_2.54mm:PinHeader_1x11_P2.54mm_Vertical -> Connector_PinHeader_2.54mm:PinHeader_1x12_P2.54mm_Vertical
- R2: value 100k -> 10k
- moved R2 3.31 mm to (100.5, 129.8), turned to 270 degrees
- moved J2 1.46 mm to (89.8, 132.5)
- moved C3 1.25 mm to (104.2, 127.8)
Connections:
- J2 pad 1: /VCC -> /EN
- J2 pad 10: /BUSY -> /RST
- J2 pad 11: /RAM_CS -> /BUSY
- J2 pad 2: /GND -> /VCC
- J2 pad 3: /MISO -> /GND
- J2 pad 4: /SD_CS -> /MISO
- J2 pad 5: /MOSI -> /SD_CS
- J2 pad 6: /SCLK -> /MOSI
- J2 pad 7: /E_CS -> /SCLK
- J2 pad 8: /DC -> /E_CS
- J2 pad 9: /RST -> /DC
- R2 pad 2: /GND -> /EN
- U2 pad 3: /VCC -> /EN
Routing:
- net /EN: track 0.00 -> 20.7 mm
- net /VCC: track 68.5 -> 64.8 mm
- net /MOSI: track 27.9 -> 26.6 mm
- net /MISO: track 38.5 -> 37.2 mm
- net /SD_CS: track 18.7 -> 17.4 mm
- net /GND: track 14.1 -> 15.0 mm
Other:
- board text added: "EN"
