File: Case/Edgework/SerialNumber/ECAD/EPaperDriver.sch (KiCad schematic (older format))
At the start: 28 parts, among them J1 Micro_SD_Card_Det, J2 Conn_01x11, Q1 Si1304BDL, U1 TXS0108EPW, U2 RT9193-33GB, U3 23LC1024

Commit message: Moved some files into correct subfolder
Parts:
- removed J2: Conn_01x11, Connector_PinHeader_2.54mm:PinHeader_1x11_P2.54mm_Vertical, symbol Connector_Generic:Conn_01x11
- added J2: Conn_01x12, Connector_PinHeader_2.54mm:PinHeader_1x12_P2.54mm_Vertical, symbol Connector_Generic:Conn_01x12
- R2: value 100k -> 10k
Connections:
- net labels added: EN
- wire segments 129 -> 128
Changed lines of the file:
@@
 $EndComp
 Wire Wire Line
-	2200 7100 2100 7100
-Wire Wire Line
-	2200 7000 2100 7000
-Wire Wire Line
-	2200 6900 2100 6900
-Wire Wire Line
-	2200 6800 2100 6800
-Wire Wire Line
-	2200 6700 2100 6700
-Wire Wire Line
-	2200 6600 2100 6600
-Wire Wire Line
-	2200 6300 2100 6300
-Wire Wire Line
-	2200 6200 2100 6200
-Text Label 2200 6200 0    50   ~ 0
-VCC
-Text Label 2200 6300 0    50   ~ 0
-GND
-Text Label 2200 6600 0    50   ~ 0
+	2300 7100 2200 7100
+Wire Wire Line
+	2300 7000 2200 7000
+Wire Wire Line
+	2300 6900 2200 6900
+Wire Wire Line
+	2300 6800 2200 6800
+Wire Wire Line
+	2300 6700 2200 6700
+Wire Wire Line
+	2300 6600 2200 6600
+Wire Wire Line
+	2300 6300 2200 6300
+Text Label 2300 6300 0    50   ~ 0
+GND
+Text Label 2300 6600 0    50   ~ 0
 MOSI
-Text Label 2200 6700 0    50   ~ 0
+Text Label 2300 6700 0    50   ~ 0
 SCLK
-Text Label 2200 6800 0    50   ~ 0
+Text Label 2300 6800 0    50   ~ 0
 E_CS
-Text Label 2200 6900 0    50   ~ 0
+Text Label 2300 6900 0    50   ~ 0
 DC
-Text Label 2200 7000 0    50   ~ 0
+Text Label 2300 7000 0    50   ~ 0
 RST
-Text Label 2200 7100 0    50   ~ 0
+Text Label 2300 7100 0    50   ~ 0
 BUSY
 Wire Wire Line
@@
 Wire Wire Line
 	5050 1600 5150 1600
-Text Label 1400 4350 2    50   ~ 0
+Text Label 1400 4300 2    50   ~ 0
 VCC
 Text Label 2600 4300 0    50   ~ 0
@@
 P 1500 4550
 F 0 "R2" H 1568 4596 50  0000 L CNN
-F 1 "100k" H 1568 4505 50  0000 L CNN
+F 1 "10k" H 1568 4505 50  0000 L CNN
 F 2 "Resistor_SMD:R_0805_2012Metric_Pad1.15x1.40mm_HandSolder" V 1540 4540 50  0001 C CNN
 F 3 "~" H 1500 4550 50  0001 C CNN
 	1    1500 4550
-	1    0    0    -1
+	-1   0    0    1
 $EndComp
 Wire Wire Line
@@
 Wire Wire Line
 	1700 4400 1500 4400
-Wire Wire Line
-	1500 4700 1500 4800
 $Comp
 L Device:C C3
@@
 	2450 4800 2450 4700
 Wire Wire Line
-	1500 4800 2000 4800
-Wire Wire Line
 	2000 4800 2450 4800
 Connection ~ 2000 4800
@@
 Wire Wire Line
 	2000 3900 2450 3900
-Wire Wire Line
-	1500 4300 1500 4350
-Connection ~ 1500 4300
-Connection ~ 1500 4400
-Wire Wire Line
-	1500 4350 1400 4350
-Connection ~ 1500 4350
-Wire Wire Line
-	1500 4350 1500 4400
 Text Label 2450 2350 0    50   ~ 0
 BS
@@
 	1    0    0    -1
 $EndComp
-$Comp
-L Connector_Generic:Conn_01x11 J2
-U 1 1 5F91087B
-P 1900 6700
-F 0 "J2" H 1818 5975 50  0000 C CNN
-F 1 "Conn_01x11" H 1818 6066 50  0000 C CNN
-F 2 "Connector_PinHeader_2.54mm:PinHeader_1x11_P2.54mm_Vertical" H 1900 6700 50  0001 C CNN
-F 3 "~" H 1900 6700 50  0001 C CNN
-	1    1900 6700
-	-1   0    0    -1
-$EndComp
-Wire Wire Line
-	2200 6400 2100 6400
-Text Label 2200 6400 0    50   ~ 0
+Wire Wire Line
+	2300 6400 2200 6400
+Text Label 2300 6400 0    50   ~ 0
 MISO
 Wire Wire Line
@@
 MISO'
 Wire Wire Line
-	2200 6500 2100 6500
-Text Label 2200 6500 0    50   ~ 0
+	2300 6500 2200 6500
+Text Label 2300 6500 0    50   ~ 0
 SD_CS
 Wire Wire Line
-	2200 7200 2100 7200
-Text Label 2200 7200 0    50   ~ 0
+	2300 7200 2200 7200
+Text Label 2300 7200 0    50   ~ 0
 RAM_CS
 Wire Wire Line
@@
 Text Label 6750 4600 0    50   ~ 0
 GND
+Wire Wire Line
+	1500 4300 1400 4300
+Connection ~ 1500 4300
+Text Label 1500 4800 0    50   ~ 0
+VCC
+Wire Wire Line
+	1500 4800 1500 4700
+Wire Wire Line
+	1500 4400 1400 4400
+Connection ~ 1500 4400
+Text Label 1400 4400 2    50   ~ 0
+EN
+$Comp
+L Connector_Generic:Conn_01x12 J2
+U 1 1 5F9569D9
+P 2000 6600
+F 0 "J2" H 1918 7317 50  0000 C CNN
+F 1 "Conn_01x12" H 1918 7226 50  0000 C CNN
+F 2 "Connector_PinHeader_2.54mm:PinHeader_1x12_P2.54mm_Vertical" H 2000 6600 50  0001 C CNN
+F 3 "~" H 2000 6600 50  0001 C CNN
+	1    2000 6600
+	-1   0    0    -1
+$EndComp
+Text Label 2300 6200 0    50   ~ 0
+VCC
+Wire Wire Line
+	2300 6200 2200 6200
+Text Label 2300 6100 0    50   ~ 0
+EN
+Wire Wire Line
+	2300 6100 2200 6100
 $EndSCHEMATC

Commit message: Updated EPaper driver
Parts:
- FPC1: symbol Display_Graphic:MDE029A128296RBW -> EPaperDriver-rescue:MDE029A128296RBW-Display_Graphic-EPaperDriver-rescue
- U3: symbol Memory_RAM:23LC1024 -> EPaperDriver-rescue:23LC1024-Memory_RAM-EPaperDriver-rescue
Changed lines of the file:
@@
 EESchema Schematic File Version 4
-LIBS:EPaperDriver-cache
-EELAYER 29 0
+EELAYER 30 0
 EELAYER END
 $Descr A4 11693 8268
@@
 3V3 = 3-line SPI
 $Comp
-L Display_Graphic:MDE029A128296RBW FPC1
+L EPaperDriver-rescue:MDE029A128296RBW-Display_Graphic-EPaperDriver-rescue FPC1
 U 1 1 5F899E8A
 P 10050 1050
@@
 	9750 5500 9750 5300
 $Comp
-L Memory_RAM:23LC1024 U3
+L EPaperDriver-rescue:23LC1024-Memory_RAM-EPaperDriver-rescue U3
 U 1 1 5F90D53F
 P 5300 6200
