File: Case/Edgework/ECAD/EdgeWorkController.sch (KiCad schematic (older format))
At the start: 31 parts, among them J1 comm_header, J2 prog_header, J3 Epaper Display, J5 Widget_2, J6 Widget_3, J7 Widget_4, J8 Widget_5, J9 Conn_01x04, U1 ATmega328-PU, U2 MCP3008

Commit message: Update a bunch of stuff
Parts:
- added SW1: SW_Push_Dual, symbol Switch:SW_Push_Dual
- gave numbers to parts that had none: 15
Connections:
- net GND: now also SW1.2
- net rst: now also SW1.1
- no-connect marks 8 -> 14
Changed lines of the file:
@@
 $EndComp
-Wire Wire Line
-	2200 2400 2200 2300
 Wire Wire Line
 	2200 2000 2200 1900
@@
 $EndComp
 $Comp
-L Connector_Generic:Conn_01x04 J?
+L Connector_Generic:Conn_01x04 J10
 U 1 1 60B6F7C7
 P 9400 2900
-F 0 "J?" V 9272 3080 50  0000 L CNN
+F 0 "J10" V 9272 3080 50  0000 L CNN
 F 1 "Conn_01x04" V 9363 3080 50  0000 L CNN
 F 2 "" H 9400 2900 50  0001 C CNN
@@
 	10250 3250 10250 3050
 $Comp
-L Device:R_US R?
+L Device:R_US R14
 U 1 1 60B6F7DD
 P 10250 2900
-F 0 "R?" H 10318 2946 50  0000 L CNN
+F 0 "R14" H 10318 2946 50  0000 L CNN
 F 1 "10k" H 10318 2855 50  0000 L CNN
 F 2 "" V 10290 2890 50  0001 C CNN
@@
 $EndComp
 $Comp
-L Connector_Generic:Conn_01x04 J?
+L Connector_Generic:Conn_01x04 J11
 U 1 1 60B845FB
 P 9400 4000
-F 0 "J?" V 9272 4180 50  0000 L CNN
+F 0 "J11" V 9272 4180 50  0000 L CNN
 F 1 "Conn_01x04" V 9363 4180 50  0000 L CNN
 F 2 "" H 9400 4000 50  0001 C CNN
@@
 	10250 4350 10250 4150
 $Comp
-L Device:R_US R?
+L Device:R_US R15
 U 1 1 60B84611
 P 10250 4000
-F 0 "R?" H 10318 4046 50  0000 L CNN
+F 0 "R15" H 10318 4046 50  0000 L CNN
 F 1 "5k" H 10318 3955 50  0000 L CNN
 F 2 "" V 10290 3990 50  0001 C CNN
@@
 $EndComp
 $Comp
-L Device:R_US R?
+L Device:R_US R10
 U 1 1 60C9D19C
 P 8050 2450
-F 0 "R?" V 8100 2300 50  0000 L CNN
+F 0 "R10" V 8100 2300 50  0000 L CNN
 F 1 "10k" V 7950 2400 50  0000 L CNN
 F 2 "" V 8090 2440 50  0001 C CNN
@@
 $EndComp
 $Comp
-L power:VCC #PWR?
+L power:VCC #PWR011
 U 1 1 60C9D1A2
 P 7850 2450
-F 0 "#PWR?" H 7850 2300 50  0001 C CNN
+F 0 "#PWR011" H 7850 2300 50  0001 C CNN
 F 1 "VCC" V 7868 2577 50  0000 L CNN
 F 2 "" H 7850 2450 50  0001 C CNN
@@
 	7900 2450 7850 2450
 $Comp
-L Device:R_US R?
+L Device:R_US R11
 U 1 1 60CA1D19
 P 8050 3400
-F 0 "R?" V 8100 3250 50  0000 L CNN
+F 0 "R11" V 8100 3250 50  0000 L CNN
 F 1 "10k" V 7950 3350 50  0000 L CNN
 F 2 "" V 8090 3390 50  0001 C CNN
@@
 $EndComp
 $Comp
-L power:VCC #PWR?
+L power:VCC #PWR012
 U 1 1 60CA1D1F
 P 7850 3400
-F 0 "#PWR?" H 7850 3250 50  0001 C CNN
+F 0 "#PWR012" H 7850 3250 50  0001 C CNN
 F 1 "VCC" V 7868 3527 50  0000 L CNN
 F 2 "" H 7850 3400 50  0001 C CNN
@@
 	7900 3400 7850 3400
 $Comp
-L Device:R_US R?
+L Device:R_US R12
 U 1 1 60CD0D0C
 P 8050 4350
-F 0 "R?" V 8100 4200 50  0000 L CNN
+F 0 "R12" V 8100 4200 50  0000 L CNN
 F 1 "10k" V 7950 4300 50  0000 L CNN
 F 2 "" V 8090 4340 50  0001 C CNN
@@
 $EndComp
 $Comp
-L power:VCC #PWR?
+L power:VCC #PWR013
 U 1 1 60CD0D12
 P 7850 4350
-F 0 "#PWR?" H 7850 4200 50  0001 C CNN
+F 0 "#PWR013" H 7850 4200 50  0001 C CNN
 F 1 "VCC" V 7868 4477 50  0000 L CNN
 F 2 "" H 7850 4350 50  0001 C CNN
@@
 	7900 4350 7850 4350
 $Comp
-L Device:R_US R?
+L Device:R_US R13
 U 1 1 60CD60BD
 P 8050 5300
-F 0 "R?" V 8100 5150 50  0000 L CNN
+F 0 "R13" V 8100 5150 50  0000 L CNN
 F 1 "10k" V 7950 5250 50  0000 L CNN
 F 2 "" V 8090 5290 50  0001 C CNN
@@
 $EndComp
 $Comp
-L power:VCC #PWR?
+L power:VCC #PWR014
 U 1 1 60CD60C3
 P 7850 5300
-F 0 "#PWR?" H 7850 5150 50  0001 C CNN
+F 0 "#PWR014" H 7850 5150 50  0001 C CNN
 F 1 "VCC" V 7868 5427 50  0000 L CNN
 F 2 "" H 7850 5300 50  0001 C CNN
@@
 Connection ~ 9750 1750
 $Comp
-L Connector_Generic:Conn_01x04 J?
+L Connector_Generic:Conn_01x04 J4
 U 1 1 60B3BC61
 P 8450 1150
-F 0 "J?" H 8530 1142 50  0000 L CNN
+F 0 "J4" H 8530 1142 50  0000 L CNN
 F 1 "Widget_1" H 8530 1051 50  0000 L CNN
 F 2 "" H 8450 1150 50  0001 C CNN
@@
 WIDGET_1
 $Comp
-L Device:R_US R?
+L Device:R_US R9
 U 1 1 60B3BC6A
 P 8050 1500
-F 0 "R?" V 8100 1350 50  0000 L CNN
+F 0 "R9" V 8100 1350 50  0000 L CNN
 F 1 "10k" V 7950 1450 50  0000 L CNN
 F 2 "" V 8090 1490 50  0001 C CNN
@@
 $EndComp
 $Comp
-L power:VCC #PWR?
+L power:VCC #PWR010
 U 1 1 60B3BC70
 P 7850 1500
-F 0 "#PWR?" H 7850 1350 50  0001 C CNN
+F 0 "#PWR010" H 7850 1350 50  0001 C CNN
 F 1 "VCC" V 7868 1627 50  0000 L CNN
 F 2 "" H 7850 1500 50  0001 C CNN
@@
 	7900 1500 7850 1500
 $Comp
-L power:GND #PWR?
+L power:GND #PWR015
 U 1 1 60B3BC7D
 P 8200 950
-F 0 "#PWR?" H 8200 700 50  0001 C CNN
+F 0 "#PWR015" H 8200 700 50  0001 C CNN
 F 1 "GND" H 8200 800 50  0000 C CNN
 F 2 "" H 8200 950 50  0001 C CNN
@@
 $EndComp
 $Comp
-L Device:R_US R?
+L Device:R_US R2
 U 1 1 60B3BC85
 P 8000 1050
-F 0 "R?" V 8050 900 50  0000 L CNN
+F 0 "R2" V 8050 900 50  0000 L CNN
 F 1 "10k" V 8050 1150 50  0000 L CNN
 F 2 "" V 8040 1040 50  0001 C CNN
@@
 	8200 1050 8150 1050
 $Comp
-L power:GND #PWR?
+L power:GND #PWR016
 U 1 1 60BF4981
 P 8200 1900
-F 0 "#PWR?" H 8200 1650 50  0001 C CNN
+F 0 "#PWR016" H 8200 1650 50  0001 C CNN
 F 1 "GND" H 8200 1750 50  0000 C CNN
 F 2 "" H 8200 1900 50  0001 C CNN
@@
 $EndComp
 $Comp
-L Device:R_US R?
+L Device:R_US R3
 U 1 1 60BF4987
 P 8000 2000
-F 0 "R?" V 8050 1850 50  0000 L CNN
+F 0 "R3" V 8050 1850 50  0000 L CNN
 F 1 "10k" V 8050 2100 50  0000 L CNN
 F 2 "" V 8040 1990 50  0001 C CNN
@@
 	8200 2000 8150 2000
 $Comp
-L power:GND #PWR?
+L power:GND #PWR017
 U 1 1 60BFA656
 P 8200 2850
-F 0 "#PWR?" H 8200 2600 50  0001 C CNN
+F 0 "#PWR017" H 8200 2600 50  0001 C CNN
 F 1 "GND" H 8200 2700 50  0000 C CNN
 F 2 "" H 8200 2850 50  0001 C CNN
@@
 $EndComp
 $Comp
-L Device:R_US R?
+L Device:R_US R4
 U 1 1 60BFA65C
 P 8000 2950
-F 0 "R?" V 8050 2800 50  0000 L CNN
+F 0 "R4" V 8050 2800 50  0000 L CNN
 F 1 "10k" V 8050 3050 50  0000 L CNN
 F 2 "" V 8040 2940 50  0001 C CNN
@@
 	8200 2950 8150 2950
 $Comp
-L power:GND #PWR?
+L power:GND #PWR018
 U 1 1 60C099D2
 P 8200 3800
-F 0 "#PWR?" H 8200 3550 50  0001 C CNN
+F 0 "#PWR018" H 8200 3550 50  0001 C CNN
 F 1 "GND" H 8200 3650 50  0000 C CNN
 F 2 "" H 8200 3800 50  0001 C CNN
@@
 $EndComp
 $Comp
-L Device:R_US R?
+L Device:R_US R5
 U 1 1 60C099D8
 P 8000 3900
-F 0 "R?" V 8050 3750 50  0000 L CNN
+F 0 "R5" V 8050 3750 50  0000 L CNN
 F 1 "10k" V 8050 4000 50  0000 L CNN
 F 2 "" V 8040 3890 50  0001 C CNN
@@
 	8200 3900 8150 3900
 $Comp
-L power:GND #PWR?
+L power:GND #PWR019
 U 1 1 60C18145
 P 8200 4750
-F 0 "#PWR?" H 8200 4500 50  0001 C CNN
+F 0 "#PWR019" H 8200 4500 50  0001 C CNN
 F 1 "GND" H 8200 4600 50  0000 C CNN
 F 2 "" H 8200 4750 50  0001 C CNN
@@
 $EndComp
 $Comp
-L Device:R_US R?
+L Device:R_US R6
 U 1 1 60C1814B
 P 8000 4850
-F 0 "R?" V 8050 4700 50  0000 L CNN
+F 0 "R6" V 8050 4700 50  0000 L CNN
 F 1 "10k" V 8050 4950 50  0000 L CNN
 F 2 "" V 8040 4840 50  0001 C CNN
@@
 Wire Wire Line
 	7800 2100 8250 2100
+$Comp
+L Switch:SW_Push_Dual SW1
+U 1 1 60F8CA14
+P 2800 1350
+F 0 "SW1" H 2800 1635 50  0000 C CNN
+F 1 "SW_Push_Dual" H 2800 1544 50  0000 C CNN
+F 2 "" H 2800 1550 50  0001 C CNN
+F 3 "~" H 2800 1550 50  0001 C CNN
+	1    2800 1350
+	1    0    0    -1
+$EndComp
+Wire Wire Line
+	2200 2300 2200 2400
+$Comp
+L power:GND #PWR03
+U 1 1 60F93BE7
+P 3100 1350
+F 0 "#PWR03" H 3100 1100 50  0001 C CNN
+F 1 "GND" H 3105 1177 50  0000 C CNN
+F 2 "" H 3100 1350 50  0001 C CNN
+F 3 "" H 3100 1350 50  0001 C CNN
+	1    3100 1350
+	0    -1   -1   0
+$EndComp
+Text Label 2500 1350 2    50   ~ 0
+rst
+Wire Wire Line
+	2500 1350 2600 1350
+Wire Wire Line
+	3000 1350 3100 1350
+NoConn ~ 3000 1550
+NoConn ~ 2600 1550
+NoConn ~ 9600 2800
+NoConn ~ 9600 2900
+NoConn ~ 9600 3900
+NoConn ~ 9600 4000
 $EndSCHEMATC
