File: Modules/NeedyCapacitorDischarge/ECAD/NeedyCapacitorDischarge.sch (KiCad schematic (older format))
At the start: 18 parts, among them J1 comm_header, J2 prog_header, SW1 SW_Push_Dual_x2, U1 ATmega328-PU, U2 MAX7219, U3 LTD6640E

Commit message: Added polyfuses to all modules
Parts:
- added F1: Polyfuse, symbol Device:Polyfuse
Connections:
- net VCC: now also F1.1; no longer J1.4 (Pin_4), J2.1 (Pin_1)
- new net UVCC: F1.2, J1.4 (Pin_4), J2.1 (Pin_1)
Changed lines of the file:
@@
 L power:VCC #PWR01
 U 1 1 5F5DC5B2
-P 1400 3350
-F 0 "#PWR01" H 1400 3200 50  0001 C CNN
-F 1 "VCC" V 1418 3477 50  0000 L CNN
-F 2 "" H 1400 3350 50  0001 C CNN
-F 3 "" H 1400 3350 50  0001 C CNN
-	1    1400 3350
-	0    -1   -1   0
-$EndComp
-$Comp
-L power:VCC #PWR03
-U 1 1 5F5DD568
-P 1400 3950
-F 0 "#PWR03" H 1400 3800 50  0001 C CNN
-F 1 "VCC" V 1418 4077 50  0000 L CNN
-F 2 "" H 1400 3950 50  0001 C CNN
-F 3 "" H 1400 3950 50  0001 C CNN
-	1    1400 3950
-	0    -1   -1   0
+P 2150 3000
+F 0 "#PWR01" H 2150 2850 50  0001 C CNN
+F 1 "VCC" V 2168 3127 50  0000 L CNN
+F 2 "" H 2150 3000 50  0001 C CNN
+F 3 "" H 2150 3000 50  0001 C CNN
+	1    2150 3000
+	0    1    1    0
 $EndComp
 $Comp
@@
 NoConn ~ 4400 4150
 NoConn ~ 4400 4050
+$Comp
+L Device:Polyfuse F1
+U 1 1 5F9289D4
+P 1900 3000
+F 0 "F1" V 1675 3000 50  0000 C CNN
+F 1 "Polyfuse" V 1766 3000 50  0000 C CNN
+F 2 "" H 1950 2800 50  0001 L CNN
+F 3 "~" H 1900 3000 50  0001 C CNN
+	1    1900 3000
+	0    1    1    0
+$EndComp
+Text Label 1400 3950 2    50   ~ 0
+UVCC
+Text Label 1400 3350 2    50   ~ 0
+UVCC
+Text Label 1650 3000 2    50   ~ 0
+UVCC
+Wire Wire Line
+	1650 3000 1750 3000
+Wire Wire Line
+	2050 3000 2150 3000
 $EndSCHEMATC

Commit message: Update a bunch of stuff
Parts:
- removed D13: Red, symbol Device:LED
- added D2: LED_RCBG, symbol Device:LED_RCBG
- added SW2: SW_Push_Dual, symbol Switch:SW_Push_Dual
- U1: symbol MCU_Microchip_ATmega:ATmega328-PU -> NeedyCapacitorDischarge-rescue:ATmega328-PU-MCU_Microchip_ATmega
Connections:
- net GND: now also D2.2 (K), SW2.2
- net rst: now also SW2.1
- net at R2.2: now also D2.1 (RA)
- no-connect marks 18 -> 22
Changed lines of the file:
@@
 EESchema Schematic File Version 4
-LIBS:NeedyCapacitorDischarge-cache
-EELAYER 29 0
+EELAYER 30 0
 EELAYER END
 $Descr A4 11693 8268
@@
 $EndDescr
 $Comp
-L MCU_Microchip_ATmega:ATmega328-PU U1
+L NeedyCapacitorDischarge-rescue:ATmega328-PU-MCU_Microchip_ATmega U1
 U 1 1 5F599BB8
 P 3800 3250
@@
 	-1   0    0    1
 $EndComp
-Wire Wire Line
-	2750 3650 2750 3750
 Wire Wire Line
 	2750 4450 2750 4550
@@
 	7000 3050 7000 4300
 NoConn ~ 6300 2050
-$Comp
-L Device:LED D13
-U 1 1 5F749B98
-P 2750 3900
-F 0 "D13" H 2743 4116 50  0000 C CNN
-F 1 "Red" H 2743 4025 50  0000 C CNN
-F 2 "" H 2750 3900 50  0001 C CNN
-F 3 "~" H 2750 3900 50  0001 C CNN
-	1    2750 3900
-	0    1    1    0
-$EndComp
 NoConn ~ 4400 4350
 $Comp
@@
 $EndComp
 Wire Wire Line
-	2750 4150 2750 4050
-Wire Wire Line
 	5500 4500 5850 4500
 NoConn ~ 4400 4250
@@
 Wire Wire Line
 	2050 3000 2150 3000
+$Comp
+L Device:LED_RCBG D2
+U 1 1 60F907FB
+P 2750 3900
+F 0 "D2" V 2704 4260 50  0000 L CNN
+F 1 "LED_RCBG" V 2795 4260 50  0000 L CNN
+F 2 "" H 2750 3850 50  0001 C CNN
+F 3 "~" H 2750 3850 50  0001 C CNN
+	1    2750 3900
+	0    1    1    0
+$EndComp
+Wire Wire Line
+	2750 3700 2750 3650
+Wire Wire Line
+	2750 4150 2950 4150
+Wire Wire Line
+	2950 4150 2950 4100
+NoConn ~ 2750 4100
+NoConn ~ 2550 4100
+$Comp
+L Switch:SW_Push_Dual SW2
+U 1 1 60FCEA85
+P 2800 1350
+F 0 "SW2" H 2800 1635 50  0000 C CNN
+F 1 "SW_Push_Dual" H 2800 1544 50  0000 C CNN
+F 2 "" H 2800 1550 50  0001 C CNN
+F 3 "~" H 2800 1550 50  0001 C CNN
+	1    2800 1350
+	1    0    0    -1
+$EndComp
+$Comp
+L power:GND #PWR03
+U 1 1 60FCF4E5
+P 3100 1350
+F 0 "#PWR03" H 3100 1100 50  0001 C CNN
+F 1 "GND" H 3105 1177 50  0000 C CNN
+F 2 "" H 3100 1350 50  0001 C CNN
+F 3 "" H 3100 1350 50  0001 C CNN
+	1    3100 1350
+	0    -1   -1   0
+$EndComp
+Text Label 2500 1350 2    50   ~ 0
+rst
+Wire Wire Line
+	2500 1350 2600 1350
+Wire Wire Line
+	3000 1350 3100 1350
+NoConn ~ 3000 1550
+NoConn ~ 2600 1550
 $EndSCHEMATC
