File: Modules/Timer/ECAD/Timer.sch (KiCad schematic (older format))
At the start: 30 parts, among them J1 comm_header, J2 prog_header, U1 ATmega328-PU, U10 NodeMCU_ESP-32S, U2 KCSC02-105, U3 KCSC02-105, U4 MAX7219, U5 KCSC02-105, U6 KCSC02-105, U7 DFPLAYER_MINI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

Commit message: Update a bunch of stuff
Parts:
- removed D1: Clear_Led, symbol Device:LED
- added D1: LED_RCBG, symbol Device:LED_RCBG
- added R10: 2k, symbol Device:R_US
- added R11: 0, symbol Device:R_US
- added R9: 1k, symbol Device:R_US
- added SW1: SW_Push_Dual, symbol Switch:SW_Push_Dual
- R4: value 3.3k -> 2k
- R6: value 2.2k -> 1k
Connections:
- net GND: now also D1.2 (K), R10.1, SW1.2
- net VCC: now also U10.19 (VIN)
- net rst: now also SW1.1
- net at U1.19 (SCK/PB5): now also R11.1; no longer U7.3 (TX)
- net at U1.5 (PD3): now also R9.2; no longer U10.27 (RX2/IO16)
- net at R2.1: now also D1.4 (GA)
- new net: R11.2, U7.3 (TX)
- new net: R10.2, R9.1, U10.27 (RX2/IO16)
- no-connect marks 71 -> 74
Changed lines of the file:
@@
 $EndComp
-Wire Wire Line
-	2750 3650 2750 3750
 Wire Wire Line
 	2750 4450 2750 4550
@@
 U 1 1 5F83C518
 P 4700 6950
-F 0 "LS1" V 4617 7130 50  0000 L CNN
-F 1 "Speaker" V 4708 7130 50  0000 L CNN
+F 0 "LS1" V 4600 7050 50  0000 L CNN
+F 1 "Speaker" V 4700 7050 50  0000 L CNN
 F 2 "" H 4700 6750 50  0001 C CNN
 F 3 "~" H 4690 6900 50  0001 C CNN
@@
 	0    -1   1    0
 $EndComp
-$Comp
-L Device:LED D1
-U 1 1 5F840032
-P 2750 3900
-F 0 "D1" V 2697 3978 50  0000 L CNN
-F 1 "Clear_Led" V 2788 3978 50  0000 L CNN
-F 2 "" H 2750 3900 50  0001 C CNN
-F 3 "~" H 2750 3900 50  0001 C CNN
-	1    2750 3900
-	0    1    1    0
-$EndComp
-Wire Wire Line
-	2750 4150 2750 4050
 $Comp
 L Device:Polyfuse F1
@@
 Wire Wire Line
 	4250 4950 4250 5950
-Wire Wire Line
-	4250 5950 5050 5950
 NoConn ~ 4400 4250
 NoConn ~ 4400 4350
@@
 U 1 1 60B17B1E
 P 1800 6150
-F 0 "U10" H 1800 7531 50  0000 C CNN
-F 1 "NodeMCU_ESP-32S" H 1800 7440 50  0000 C CNN
+F 0 "U10" H 2700 7300 50  0000 C CNN
+F 1 "NodeMCU_ESP-32S" H 1150 7300 50  0000 C CNN
 F 2 "Module:NodeMCU_ESP-32S" H 1100 5000 50  0001 C CNN
 F 3 "https://einstronic.com/wp-content/uploads/2017/06/NodeMCU-32S-Catalogue.pdf" H 1800 4850 50  0001 C CNN
@@
 NoConn ~ 2900 5950
 NoConn ~ 1800 4950
-NoConn ~ 1700 4950
 Wire Wire Line
 	4400 4050 5700 4050
@@
 Wire Wire Line
 	5700 4850 4150 4850
-Wire Wire Line
-	4150 4850 4150 6850
-Wire Wire Line
-	4150 6850 2900 6850
 Wire Wire Line
 	2900 6750 4050 6750
@@
 P 5350 5050
 F 0 "R6" V 5300 5100 50  0000 L CNN
-F 1 "2.2k" V 5250 4950 50  0000 L CNN
+F 1 "1k" V 5250 4950 50  0000 L CNN
 F 2 "" V 5390 5040 50  0001 C CNN
 F 3 "~" H 5350 5050 50  0001 C CNN
@@
 P 4800 5050
 F 0 "R4" V 4750 5100 50  0000 L CNN
-F 1 "3.3k" V 4700 4950 50  0000 L CNN
+F 1 "2k" V 4700 4950 50  0000 L CNN
 F 2 "" V 4840 5040 50  0001 C CNN
 F 3 "~" H 4800 5050 50  0001 C CNN
@@
 Wire Wire Line
 	8050 2000 8950 2000
+$Comp
+L power:VCC #PWR023
+U 1 1 60CD97CA
+P 1700 4850
+F 0 "#PWR023" H 1700 4700 50  0001 C CNN
+F 1 "VCC" V 1718 4977 50  0000 L CNN
+F 2 "" H 1700 4850 50  0001 C CNN
+F 3 "" H 1700 4850 50  0001 C CNN
+	1    1700 4850
+	1    0    0    -1
+$EndComp
+Wire Wire Line
+	1700 4950 1700 4850
+$Comp
+L Device:R_US R9
+U 1 1 60E3F9BF
+P 4150 6600
+F 0 "R9" V 4100 6650 50  0000 L CNN
+F 1 "1k" V 4050 6500 50  0000 L CNN
+F 2 "" V 4190 6590 50  0001 C CNN
+F 3 "~" H 4150 6600 50  0001 C CNN
+	1    4150 6600
+	-1   0    0    1
+$EndComp
+$Comp
+L Device:R_US R10
+U 1 1 60E3F9C5
+P 4150 7100
+F 0 "R10" V 4100 7150 50  0000 L CNN
+F 1 "2k" V 4050 7000 50  0000 L CNN
+F 2 "" V 4190 7090 50  0001 C CNN
+F 3 "~" H 4150 7100 50  0001 C CNN
+	1    4150 7100
+	-1   0    0    1
+$EndComp
+Wire Wire Line
+	4150 4850 4150 6450
+Wire Wire Line
+	2900 6850 4150 6850
+Wire Wire Line
+	4150 6850 4150 6750
+Wire Wire Line
+	4150 6850 4150 6950
+Connection ~ 4150 6850
+$Comp
+L power:GND #PWR?
+U 1 1 60EA9B80
+P 4150 7350
+AR Path="/5F832F87/60EA9B80" Ref="#PWR?"  Part="1"
+AR Path="/60EA9B80" Ref="#PWR025"  Part="1"
+F 0 "#PWR025" H 4150 7100 50  0001 C CNN
+F 1 "GND" H 4155 7177 50  0000 C CNN
+F 2 "" H 4150 7350 50  0001 C CNN
+F 3 "" H 4150 7350 50  0001 C CNN
+	1    4150 7350
+	1    0    0    -1
+$EndComp
+Wire Wire Line
+	4150 7350 4150 7250
+$Comp
+L Device:R_US R11
+U 1 1 60E4138E
+P 4600 5950
+F 0 "R11" V 4550 6000 50  0000 L CNN
+F 1 "0" V 4500 5850 50  0000 L CNN
+F 2 "" V 4640 5940 50  0001 C CNN
+F 3 "~" H 4600 5950 50  0001 C CNN
+	1    4600 5950
+	0    -1   -1   0
+$EndComp
+Wire Wire Line
+	4450 5950 4250 5950
+Wire Wire Line
+	4750 5950 5050 5950
+$Comp
+L Switch:SW_Push_Dual SW1
+U 1 1 60F94066
+P 2850 1350
+F 0 "SW1" H 2850 1635 50  0000 C CNN
+F 1 "SW_Push_Dual" H 2850 1544 50  0000 C CNN
+F 2 "" H 2850 1550 50  0001 C CNN
+F 3 "~" H 2850 1550 50  0001 C CNN
+	1    2850 1350
+	1    0    0    -1
+$EndComp
+$Comp
+L power:GND #PWR024
+U 1 1 60F95311
+P 3150 1350
+F 0 "#PWR024" H 3150 1100 50  0001 C CNN
+F 1 "GND" H 3155 1177 50  0000 C CNN
+F 2 "" H 3150 1350 50  0001 C CNN
+F 3 "" H 3150 1350 50  0001 C CNN
+	1    3150 1350
+	0    -1   -1   0
+$EndComp
+Text Label 2550 1350 2    50   ~ 0
+rst
+Wire Wire Line
+	2550 1350 2650 1350
+NoConn ~ 3050 1550
+NoConn ~ 2650 1550
+$Comp
+L Device:LED_RCBG D1
+U 1 1 60FC33EF
+P 2750 3900
+F 0 "D1" V 2704 4260 50  0000 L CNN
+F 1 "LED_RCBG" V 2795 4260 50  0000 L CNN
+F 2 "" H 2750 3850 50  0001 C CNN
+F 3 "~" H 2750 3850 50  0001 C CNN
+	1    2750 3900
+	0    1    1    0
+$EndComp
+Wire Wire Line
+	2750 3700 2750 3650
+Wire Wire Line
+	2750 4150 2750 4100
+NoConn ~ 2950 4100
+NoConn ~ 2550 4100
+Wire Wire Line
+	3050 1350 3150 1350
 $EndSCHEMATC
